File: INA219.kicad_sch (KiCad schematic)
At the start: 21 parts, among them Q1 IRFZ44N, Q2 IRFZ44N, Q3 IRFZ44N, U2 INA219AxD, U5 INA219AxD, U6 INA219AxD

Commit message: v1
Parts:
- removed Q1, Q2, Q3: IRFZ44N, Package_TO_SOT_THT:TO-220-3_Horizontal_TabDown, symbol IRFZ44N:IRFZ44N
- removed R10, R2, R3, R5, R6, R9: 10K, Resistor_SMD:R_0805_2012Metric_Pad1.20x1.40mm_HandSolder, symbol Device:R_US
- added Q1, Q2, Q3: IRLZ24, Package_TO_SOT_THT:TO-220-3_Horizontal_TabDown, symbol Transistor_FET:IRLZ24
- added R15, R16, R17: R_US, Resistor_THT:R_Axial_DIN0207_L6.3mm_D2.5mm_P15.24mm_Horizontal, symbol Device:R_US
Connections:
- net 3.3V_{1}: now also U2.1 (A1), U2.2 (A0); no longer U5.1 (A1), U6.2 (A0)
- net G1: now also R11.1; no longer R4.1
- net G3: now also R4.1; no longer R11.1
- net GND: now also U6.1 (A1), U6.2 (A0), Q1.3 (S), Q2.3 (S), Q3.3 (S)
- net SDA: now also U5.1 (A1), U5.2 (A0)
- net V_{in2}: now also R15.1, R16.1, R17.1; no longer R1.1, R12.1, R8.1, U2.8 (IN+), U5.8 (IN+), U6.8 (IN+)
- net at R1.2, U2.7 (IN-): now also Q1.2 (D)
- net at C10.1, R7.2: now also Q3.1 (G)
- net at R8.2, U5.7 (IN-): now also Q3.2 (D)
- net at C9.1, R4.2: now also Q1.1 (G)
- net at R12.2, U6.7 (IN-): now also Q2.2 (D)
- net at C11.1, R11.2: now also Q2.1 (G)
- new net: R1.1, R16.2, U2.8 (IN+)
- new net: R15.2, R8.1, U5.8 (IN+)
- new net: R12.1, R17.2, U6.8 (IN+)
Other:
- moved on the sheet: C10, C11, C9, R11, R4, R7
