File: espSAT.kicad_sch (KiCad schematic)
At the start: 22 parts, among them J1 Micro_SD_Card_Det2, J2 Prog, J3 C5, J4 C1, J5 C2, J6 C6, U1 ESP32-WROOM-32, U3 AZ1117-3.3, U4 AZ1117-3.3

Commit message: v1
Parts:
- removed C2: 10μF, Capacitor_SMD:C_0805_2012Metric_Pad1.18x1.45mm_HandSolder, symbol Device:C_Polarized
- removed C3: 22μF, Capacitor_SMD:C_0805_2012Metric_Pad1.18x1.45mm_HandSolder, symbol Device:C_Polarized
- J2: footprint Connector_Molex:Molex_SPOX_5267-06A_1x06_P2.50mm_Vertical -> Connector_PinSocket_2.54mm:PinSocket_1x06_P2.54mm_Horizontal
- J3, J6: footprint Connector_JST:JST_EH_B4B-EH-A_1x04_P2.50mm_Vertical -> Connector_PinSocket_1.27mm:PinSocket_1x04_P1.27mm_Vertical
- J4, J5: footprint Connector_JST:JST_EH_B2B-EH-A_1x02_P2.50mm_Vertical -> Connector_PinSocket_1.27mm:PinSocket_1x02_P1.27mm_Vertical
Connections:
- net 3.3V_{1}: now also J2.2 (Pin_2); no longer J2.6 (Pin_6)
- net DIR: now also U1.11 (IO26); no longer U1.12 (IO27)
- net IO0: now also J2.4 (Pin_4); no longer J2.2 (Pin_2)
- net STEP: now also U1.12 (IO27); no longer U1.11 (IO26)
- net TXD0: now also J2.6 (Pin_6); no longer J2.4 (Pin_4)

Commit message: v1.2
Connections:
- net G1: now also U1.28 (IO17); no longer U1.26 (IO4)
- net G3: now also U1.26 (IO4); no longer U1.28 (IO17)
Changed lines of the file:
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@@
 	(global_label "G3"
 		(shape output)
-		(at 88.9 134.62 0)
+		(at 88.9 116.84 0)
 		(fields_autoplaced yes)
 		(effects
@@
 		)
 		(property "Intersheetrefs" "${INTERSHEET_REFS}"
-			(at 94.3647 134.62 0)
+			(at 94.3647 116.84 0)
 			(effects
 				(font
@@
 	(global_label "G1"
 		(shape output)
-		(at 88.9 116.84 0)
+		(at 88.9 134.62 0)
 		(fields_autoplaced yes)
 		(effects
@@
 		)
 		(property "Intersheetrefs" "${INTERSHEET_REFS}"
-			(at 94.3647 116.84 0)
+			(at 94.3647 134.62 0)
 			(effects
 				(font
